Commit message: multiple tests

File: genesis/assets/urdf/simple/mixed_joints_robot.urdf (robot description, URDF)
Before this commit: robot three_cube_chain, 3 links, 2 joints
Links:
- removed link moving1
- removed link moving2
- added link prismatic_link, mass 1.0; collision box size=0.1 0.1 0.1; visual box size=0.1 0.1 0.1
- added link revolute_link, mass 1.0; collision box size=0.1 0.1 0.1; visual box size=0.1 0.1 0.1
Joints:
- removed joint joint1
- removed joint joint2
- added joint prismatic_joint: type prismatic, parent revolute_link, child prismatic_link, origin xyz=0.2 0 0 rpy=0 0 0, axis 1 0 0, limit lower=-0.2 upper=0.2 effort=100 velocity=1.0
- added joint revolute_joint: type revolute, parent base, child revolute_link, origin xyz=0.1 0 0 rpy=0 0 0, axis 0 0 1, limit lower=-3.14 upper=3.14 effort=100 velocity=1.0

File: genesis/assets/urdf/simple/two_cube_prismatic.urdf (robot description, URDF)
Before this commit: robot two_cube_joint, 2 links, 1 joints
Joints:
- joint joint1: axis 0 1 0 -> 1 0 0; limit lower=-1.57 upper=1.57 effort=100 velocity=1.0 -> lower=-0.3 upper=0.3 effort=100 velocity=1.0; origin xyz=0.1 0 0 rpy=0 0 0 -> xyz=0.0 0 0 rpy=0 0 0; type revolute -> prismatic
