Commit message: Update bike ground

File: examples/IPC_demo/track_bike/track_bike.urdf (robot description, URDF)
Before this commit: robot track_bike, 4 links, 3 joints
Links:
- added link front_wheel, mass 0.800000; collision mesh filename=front_wheel.obj; visual mesh filename=front_wheel.glb
- added link rear_wheel, mass 0.800000; collision mesh filename=rear_wheel.obj; visual mesh filename=rear_wheel.glb
- link bike_base: mass 8.000000 -> 6.000000
Joints:
- added joint front_wheel_joint: type continuous, parent bike_base, child front_wheel, origin xyz=0.5380368232727051 0.36400002241134644 0 rpy=0 0 0, axis 0.0 0.0 1.0
- added joint rear_wheel_joint: type fixed, parent rear_sprocket, child rear_wheel, origin xyz=0 0 -0.045414417050778866 rpy=0 0 0
- joint front_sprocket_joint: limit lower=-1e16 upper=1e16 effort=100 velocity=100 -> (none); origin xyz=-0.10924958810210228 0.31892967224121094 0.04541441705077887 rpy=0 0 0 -> xyz=-0.10924958810210228 0.31892967224121094 0.045414417050778866 rpy=0 0 0; type revolute -> continuous
- joint rear_sprocket_joint: limit lower=-1e16 upper=1e16 effort=100 velocity=100 -> (none); origin xyz=-0.5371130406856537 0.3666304647922516 0.04541441705077887 rpy=0 0 0 -> xyz=-0.5371130406856537 0.3666304647922516 0.045414417050778866 rpy=0 0 0; type revolute -> continuous
