Commit message: Update bike

File: DemoAssets/track_bike/track_bike.urdf (robot description, URDF)
Before this commit: robot track_bike, 6 links, 5 joints
Links:
- link front_sprocket: geometry collision mesh filename=front_sprocket.obj scale=0.985 0.985 0.985; visual mesh filename=front_sprocket.glb scale=0.985 0.985 0.985
- link rear_sprocket: geometry collision mesh filename=rear_sprocket.obj scale=0.985 0.985 0.985; visual mesh filename=rear_sprocket.glb scale=0.985 0.985 0.985
