Commit message: Visual fixes to sharpa hand urdf

File: DemoAssets/marvin_sharpa_description/marvin_sharpa.urdf (robot description, URDF)
Before this commit: robot bimanual_marvin_with_sharpa_hands, 88 links, 87 joints
Links:
- link left_hand_C_MC: geometry collision mesh filename=hands/sharpa/left/meshes/left_hand_C_MC.glb; visual mesh filename=hands/sharpa/left/meshes/left_hand_C_MC_visual.glb
- link left_hand_flange: geometry visual mesh filename=hands/sharpa/left/meshes/flange_B.glb
- link left_hand_wrist: geometry collision mesh filename=hands/sharpa/left/meshes/wrist_collision.glb; visual mesh filename=hands/sharpa/left/meshes/wrist_B.glb
- link left_index_DP: geometry collision mesh filename=hands/sharpa/left/meshes/DP_HB1_4F.glb; visual mesh filename=hands/sharpa/left/meshes/DP_visual_HB1_4F.glb
- link left_index_MCP_VL: geometry collision mesh filename=hands/sharpa/left/meshes/MCP_VL.glb; visual mesh filename=hands/sharpa/left/meshes/left_MCP_VL_visual.glb
- link left_index_MP: geometry collision mesh filename=hands/sharpa/left/meshes/left_MP.glb; visual mesh filename=hands/sharpa/left/meshes/left_MP_visual.glb
- link left_index_PP: geometry collision mesh filename=hands/sharpa/left/meshes/left_PP_mod.glb; visual mesh filename=hands/sharpa/left/meshes/left_PP_visual.glb
- link left_index_elastomer: geometry collision mesh filename=hands/sharpa/left/meshes/elastomer_HB1_4F.glb; visual mesh filename=hands/sharpa/left/meshes/elastomer_HB1_4F.glb
- link left_middle_DP: geometry collision mesh filename=hands/sharpa/left/meshes/DP_HB1_4F.glb; visual mesh filename=hands/sharpa/left/meshes/DP_visual_HB1_4F.glb
- link left_middle_MCP_VL: geometry collision mesh filename=hands/sharpa/left/meshes/MCP_VL.glb; visual mesh filename=hands/sharpa/left/meshes/left_MCP_VL_visual.glb
- link left_middle_MP: geometry collision mesh filename=hands/sharpa/left/meshes/left_MP.glb; visual mesh filename=hands/sharpa/left/meshes/left_MP_visual.glb
- link left_middle_PP: geometry collision mesh filename=hands/sharpa/left/meshes/left_PP.glb; visual mesh filename=hands/sharpa/left/meshes/left_PP_visual.glb
- link left_middle_elastomer: geometry collision mesh filename=hands/sharpa/left/meshes/elastomer_HB1_4F.glb; visual mesh filename=hands/sharpa/left/meshes/elastomer_HB1_4F.glb
- link left_pinky_DP: geometry collision mesh filename=hands/sharpa/left/meshes/DP_HB1_4F.glb; visual mesh filename=hands/sharpa/left/meshes/DP_visual_HB1_4F.glb
- link left_pinky_MC: geometry collision mesh filename=hands/sharpa/left/meshes/left_pinky_MC.glb; visual mesh filename=hands/sharpa/left/meshes/left_pinky_MC_visual.glb
- link left_pinky_MCP_VL: geometry collision mesh filename=hands/sharpa/left/meshes/MCP_VL.glb; visual mesh filename=hands/sharpa/left/meshes/left_MCP_VL_visual.glb
- link left_pinky_MP: geometry collision mesh filename=hands/sharpa/left/meshes/left_MP.glb; visual mesh filename=hands/sharpa/left/meshes/left_MP_visual.glb
- link left_pinky_PP: geometry collision mesh filename=hands/sharpa/left/meshes/left_PP.glb; visual mesh filename=hands/sharpa/left/meshes/left_PP_visual.glb
- link left_pinky_elastomer: geometry collision mesh filename=hands/sharpa/left/meshes/elastomer_HB1_4F.glb; visual mesh filename=hands/sharpa/left/meshes/elastomer_HB1_4F.glb
- link left_ring_DP: geometry collision mesh filename=hands/sharpa/left/meshes/DP_HB1_4F.glb; visual mesh filename=hands/sharpa/left/meshes/DP_visual_HB1_4F.glb
- link left_ring_MCP_VL: geometry collision mesh filename=hands/sharpa/left/meshes/MCP_VL.glb; visual mesh filename=hands/sharpa/left/meshes/left_MCP_VL_visual.glb
- link left_ring_MP: geometry collision mesh filename=hands/sharpa/left/meshes/left_MP.glb; visual mesh filename=hands/sharpa/left/meshes/left_MP_visual.glb
- link left_ring_PP: geometry collision mesh filename=hands/sharpa/left/meshes/left_PP.glb; visual mesh filename=hands/sharpa/left/meshes/left_PP_visual.glb
- link left_ring_elastomer: geometry collision mesh filename=hands/sharpa/left/meshes/elastomer_HB1_4F.glb; visual mesh filename=hands/sharpa/left/meshes/elastomer_HB1_4F.glb
- link left_thumb_CMC_VL: geometry visual mesh filename=hands/sharpa/left/meshes/left_thumb_CMC_VL.glb
- link left_thumb_DP: geometry collision mesh filename=hands/sharpa/left/meshes/DP_HB1_TH.glb; visual mesh filename=hands/sharpa/left/meshes/DP_Visual_HB1_TH.glb
- link left_thumb_MC: geometry collision mesh filename=hands/sharpa/left/meshes/left_thumb_MC.glb; visual mesh filename=hands/sharpa/left/meshes/left_thumb_MC_visual.glb
- link left_thumb_MCP_VL: geometry visual mesh filename=hands/sharpa/left/meshes/left_thumb_MCP_VL_visual.glb
- link left_thumb_PP: geometry collision mesh filename=hands/sharpa/left/meshes/left_thumb_PP.glb; visual mesh filename=hands/sharpa/left/meshes/left_thumb_PP_visual.glb
- link left_thumb_elastomer: geometry collision mesh filename=hands/sharpa/left/meshes/elastomer_HB1_TH.glb; visual mesh filename=hands/sharpa/left/meshes/elastomer_HB1_TH.glb
- link right_hand_C_MC: geometry collision mesh filename=hands/sharpa/right/meshes/right_hand_C_MC.glb; visual mesh filename=hands/sharpa/right/meshes/right_hand_C_MC_visual.glb
- link right_hand_flange: geometry visual mesh filename=hands/sharpa/right/meshes/flange_B.glb
- link right_hand_wrist: geometry collision mesh filename=hands/sharpa/right/meshes/wrist_collision.glb; visual mesh filename=hands/sharpa/right/meshes/wrist_B.glb
- link right_index_DP: geometry collision mesh filename=hands/sharpa/right/meshes/DP_HB1_4F.glb; visual mesh filename=hands/sharpa/right/meshes/DP_visual_HB1_4F.glb
- link right_index_MCP_VL: geometry collision mesh filename=hands/sharpa/right/meshes/MCP_VL.glb; visual mesh filename=hands/sharpa/right/meshes/right_MCP_VL_visual.glb
- link right_index_MP: geometry collision mesh filename=hands/sharpa/right/meshes/right_MP.glb; visual mesh filename=hands/sharpa/right/meshes/right_MP_visual.glb
- link right_index_PP: geometry collision mesh filename=hands/sharpa/right/meshes/right_PP.glb; visual mesh filename=hands/sharpa/right/meshes/right_PP_visual.glb
- link right_index_elastomer: geometry collision mesh filename=hands/sharpa/right/meshes/elastomer_HB1_4F.glb; visual mesh filename=hands/sharpa/right/meshes/elastomer_HB1_4F.glb
- link right_middle_DP: geometry collision mesh filename=hands/sharpa/right/meshes/DP_HB1_4F.glb; visual mesh filename=hands/sharpa/right/meshes/DP_visual_HB1_4F.glb
- link right_middle_MCP_VL: geometry collision mesh filename=hands/sharpa/right/meshes/MCP_VL.glb; visual mesh filename=hands/sharpa/right/meshes/right_MCP_VL_visual.glb
- link right_middle_MP: geometry collision mesh filename=hands/sharpa/right/meshes/right_MP.glb; visual mesh filename=hands/sharpa/right/meshes/right_MP_visual.glb
- link right_middle_PP: geometry collision mesh filename=hands/sharpa/right/meshes/right_PP.glb; visual mesh filename=hands/sharpa/right/meshes/right_PP_visual.glb
- link right_middle_elastomer: geometry collision mesh filename=hands/sharpa/right/meshes/elastomer_HB1_4F.glb; visual mesh filename=hands/sharpa/right/meshes/elastomer_HB1_4F.glb
- link right_pinky_DP: geometry collision mesh filename=hands/sharpa/right/meshes/DP_HB1_4F.glb; visual mesh filename=hands/sharpa/right/meshes/DP_visual_HB1_4F.glb
- link right_pinky_MC: geometry collision mesh filename=hands/sharpa/right/meshes/right_pinky_MC.glb; visual mesh filename=hands/sharpa/right/meshes/right_pinky_MC_visual.glb
- link right_pinky_MCP_VL: geometry collision mesh filename=hands/sharpa/right/meshes/MCP_VL.glb; visual mesh filename=hands/sharpa/right/meshes/right_MCP_VL_visual.glb
- link right_pinky_MP: geometry collision mesh filename=hands/sharpa/right/meshes/right_MP.glb; visual mesh filename=hands/sharpa/right/meshes/right_MP_visual.glb
- link right_pinky_PP: geometry collision mesh filename=hands/sharpa/right/meshes/right_PP.glb; visual mesh filename=hands/sharpa/right/meshes/right_PP_visual.glb
- link right_pinky_elastomer: geometry collision mesh filename=hands/sharpa/right/meshes/elastomer_HB1_4F.glb; visual mesh filename=hands/sharpa/right/meshes/elastomer_HB1_4F.glb
- link right_ring_DP: geometry collision mesh filename=hands/sharpa/right/meshes/DP_HB1_4F.glb; visual mesh filename=hands/sharpa/right/meshes/DP_visual_HB1_4F.glb
- link right_ring_MCP_VL: geometry collision mesh filename=hands/sharpa/right/meshes/MCP_VL.glb; visual mesh filename=hands/sharpa/right/meshes/right_MCP_VL_visual.glb
- link right_ring_MP: geometry collision mesh filename=hands/sharpa/right/meshes/right_MP.glb; visual mesh filename=hands/sharpa/right/meshes/right_MP_visual.glb
- link right_ring_PP: geometry collision mesh filename=hands/sharpa/right/meshes/right_PP.glb; visual mesh filename=hands/sharpa/right/meshes/right_PP_visual.glb
- link right_ring_elastomer: geometry collision mesh filename=hands/sharpa/right/meshes/elastomer_HB1_4F.glb; visual mesh filename=hands/sharpa/right/meshes/elastomer_HB1_4F.glb
- link right_thumb_CMC_VL: geometry visual mesh filename=hands/sharpa/right/meshes/right_thumb_CMC_VL_visual.glb
- link right_thumb_DP: geometry collision mesh filename=hands/sharpa/right/meshes/DP_HB1_TH.glb; visual mesh filename=hands/sharpa/right/meshes/DP_Visual_HB1_TH.glb
- link right_thumb_MC: geometry collision mesh filename=hands/sharpa/right/meshes/right_thumb_MC.glb; visual mesh filename=hands/sharpa/right/meshes/right_thumb_MC_visual.glb
- link right_thumb_MCP_VL: geometry visual mesh filename=hands/sharpa/right/meshes/right_thumb_MCP_VL_visual.glb
- link right_thumb_PP: geometry collision mesh filename=hands/sharpa/right/meshes/right_thumb_PP.glb; visual mesh filename=hands/sharpa/right/meshes/right_thumb_PP_visual.glb
- link right_thumb_elastomer: geometry collision mesh filename=hands/sharpa/right/meshes/elastomer_HB1_TH.glb; visual mesh filename=hands/sharpa/right/meshes/elastomer_HB1_TH.glb

Commit message: add cooking traj

File: DemoAssets/marvin_sharpa_description/marvin_sharpa.urdf (robot description, URDF)
Before this commit: robot bimanual_marvin_with_sharpa_hands, 88 links, 87 joints
Links:
- link left_thumb_PP: geometry collision mesh filename=hands/sharpa/left/meshes/left_thumb_PP.STL; visual mesh filename=hands/sharpa/left/meshes/left_thumb_PP_visual.glb

Commit message: Rendering tweaks: per-material-slot surfaces, replay overhaul, new scene scripts and assets (#3)

File: DemoAssets/marvin_sharpa_description/marvin_sharpa.urdf (robot description, URDF)
Before this commit: robot bimanual_marvin_with_sharpa_hands, 88 links, 87 joints
Links:
- link left_thumb_PP: geometry collision mesh filename=hands/sharpa/left/meshes/left_thumb_PP.glb; visual mesh filename=hands/sharpa/left/meshes/left_thumb_PP_visual.glb
