Commit message: perf(qipc): align tape dispenser solver configuration

File: genesis/assets/qipc/tape_dispenser_v2/tape_dispenser.urdf (robot description, URDF)
Before this commit: robot tape_dispenser_v2, 6 links, 5 joints
Links:
- link Cylinder: mass 0.0433501 -> 0.02140105760
- link tape_cutter: mass 0.27 -> 0.20046402301
- link tape_wheel: mass 0.04 -> 0.08800596439

File: genesis/assets/qipc/tape_dispenser_v2/tape_dispenser_machine.urdf (robot description, URDF)
Before this commit: robot tape_dispenser_v2, 6 links, 5 joints
Links:
- link Cylinder: mass 0.0433501 -> 0.02140105760
- link tape_cutter: mass 0.27 -> 0.20046402301
- link tape_wheel: mass 0.04 -> 0.08800596439
